Commit message: Fixed RL in Gazebo

File: simulation_world/urdf/m4.urdf (robot description, URDF)
Before this commit: robot m4assembly, 23 links, 22 joints
Links:
- removed link front_realsense_gazebo
- removed link rear_realsense
- removed link rear_realsense_gazebo
- removed link rear_realsense_lens
- link base_link: mass 5.054 -> 1.054
- link front_left_wheel: mass 2.0 -> 0.447367750292981
- link front_realsense: mass 0.05 -> None; geometry 
- link front_right_wheel: mass 2.0 -> 0.447367750640603
- link rear_left_wheel: mass 2.0 -> 0.447367748033206
- link rear_right_wheel: mass 2.0 -> 0.447367750743676
Joints:
- removed joint front_realsense_gazebo_joint
- removed joint rear_realsense_gazebo_joint
- removed joint rear_realsense_joint
- removed joint rear_realsense_lens_joint
- joint front_left_leg_joint: type fixed -> revolute
- joint front_right_leg_joint: type fixed -> revolute
- joint rear_left_leg_joint: type fixed -> revolute
- joint rear_right_leg_joint: type fixed -> revolute

File: simulation_world/urdf/m4_fixed_blade.urdf (robot description, URDF)
Before this commit: robot m4assembly, 23 links, 22 joints
Links:
- removed link front_realsense_gazebo
- removed link rear_realsense
- removed link rear_realsense_gazebo
- removed link rear_realsense_lens
- link base_link: mass 5.054 -> 1.054
- link front_left_wheel: mass 2.0 -> 0.447367750292981
- link front_realsense: mass 0.05 -> None; geometry 
- link front_right_wheel: mass 2.0 -> 0.447367750640603
- link rear_left_wheel: mass 2.0 -> 0.447367748033206
- link rear_right_wheel: mass 2.0 -> 0.447367750743676
Joints:
- removed joint front_realsense_gazebo_joint
- removed joint rear_realsense_gazebo_joint
- removed joint rear_realsense_joint
- removed joint rear_realsense_lens_joint
- joint front_left_blade_joint: type continuous -> fixed
- joint front_left_leg_joint: type fixed -> revolute
- joint front_right_blade_joint: type continuous -> fixed
- joint front_right_leg_joint: type fixed -> revolute
- joint rear_left_blade_joint: type continuous -> fixed
- joint rear_left_leg_joint: type fixed -> revolute
- joint rear_right_blade_joint: type continuous -> fixed
- joint rear_right_leg_joint: type fixed -> revolute

File: simulation_world/urdf/m4_fixed_blade_hip.urdf (robot description, URDF)
Before this commit: robot m4assembly, 23 links, 22 joints
Links:
- removed link front_realsense_gazebo
- removed link rear_realsense
- removed link rear_realsense_gazebo
- removed link rear_realsense_lens
- link base_link: mass 5.054 -> 1.054
- link front_left_wheel: mass 2.0 -> 0.447367750292981
- link front_realsense: mass 0.05 -> None; geometry 
- link front_right_wheel: mass 2.0 -> 0.447367750640603
- link rear_left_wheel: mass 2.0 -> 0.447367748033206
- link rear_right_wheel: mass 2.0 -> 0.447367750743676
Joints:
- removed joint front_realsense_gazebo_joint
- removed joint rear_realsense_gazebo_joint
- removed joint rear_realsense_joint
- removed joint rear_realsense_lens_joint
- joint front_left_blade_joint: type continuous -> fixed
- joint front_left_hip_joint: type revolute -> fixed
- joint front_left_leg_joint: type fixed -> revolute
- joint front_right_blade_joint: type continuous -> fixed
- joint front_right_hip_joint: type revolute -> fixed
- joint front_right_leg_joint: type fixed -> revolute
- joint rear_left_blade_joint: type continuous -> fixed
- joint rear_left_hip_joint: type revolute -> fixed
- joint rear_left_leg_joint: type fixed -> revolute
- joint rear_right_blade_joint: type continuous -> fixed
- joint rear_right_hip_joint: type revolute -> fixed
- joint rear_right_leg_joint: type fixed -> revolute

File: simulation_world/urdf/m4_fixed_blade_hip_leg.urdf (robot description, URDF)
Before this commit: robot m4assembly, 23 links, 22 joints
Links:
- removed link front_realsense_gazebo
- removed link rear_realsense
- removed link rear_realsense_gazebo
- removed link rear_realsense_lens
- link base_link: mass 5.054 -> 1.054
- link front_left_wheel: mass 2.0 -> 0.447367750292981
- link front_realsense: mass 0.05 -> None; geometry 
- link front_right_wheel: mass 2.0 -> 0.447367750640603
- link rear_left_wheel: mass 2.0 -> 0.447367748033206
- link rear_right_wheel: mass 2.0 -> 0.447367750743676
Joints:
- removed joint front_realsense_gazebo_joint
- removed joint rear_realsense_gazebo_joint
- removed joint rear_realsense_joint
- removed joint rear_realsense_lens_joint
- joint front_left_blade_joint: type continuous -> fixed
- joint front_left_hip_joint: type revolute -> fixed
- joint front_right_blade_joint: type continuous -> fixed
- joint front_right_hip_joint: type revolute -> fixed
- joint rear_left_blade_joint: type continuous -> fixed
- joint rear_left_hip_joint: type revolute -> fixed
- joint rear_right_blade_joint: type continuous -> fixed
- joint rear_right_hip_joint: type revolute -> fixed

File: simulation_world/urdf/m4_fixed_blade_leg.urdf (robot description, URDF)
Before this commit: robot m4assembly, 23 links, 22 joints
Links:
- removed link front_realsense_gazebo
- removed link rear_realsense
- removed link rear_realsense_gazebo
- removed link rear_realsense_lens
- link base_link: mass 5.054 -> 1.054
- link front_left_wheel: mass 2.0 -> 0.447367750292981
- link front_realsense: mass 0.05 -> None; geometry 
- link front_right_wheel: mass 2.0 -> 0.447367750640603
- link rear_left_wheel: mass 2.0 -> 0.447367748033206
- link rear_right_wheel: mass 2.0 -> 0.447367750743676
Joints:
- removed joint front_realsense_gazebo_joint
- removed joint rear_realsense_gazebo_joint
- removed joint rear_realsense_joint
- removed joint rear_realsense_lens_joint
- joint front_left_blade_joint: type continuous -> fixed
- joint front_right_blade_joint: type continuous -> fixed
- joint rear_left_blade_joint: type continuous -> fixed
- joint rear_right_blade_joint: type continuous -> fixed
